File: Hardware/ThingsGate-1/ThingsGate-1.kicad_sch (KiCad schematic)
At the start: 0 parts

Commit message: schematic
Other:
- removed sheet IO
Changed lines of the file:
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@@
 	)
 	(sheet
-		(at 166.37 83.82)
+		(at 134.62 83.82)
 		(size 17.78 20.32)
 		(exclude_from_sim no)
@@
 		)
 		(property "Sheetname" "Power Harvester"
-			(at 166.37 83.1084 0)
+			(at 134.62 83.1084 0)
 			(effects
 				(font
@@
 		)
 		(property "Sheetfile" "Power_Harvester.kicad_sch"
-			(at 166.37 104.7246 0)
+			(at 134.62 104.7246 0)
 			(effects
 				(font
@@
 				)
 			)
-		)
-	)
-	(sheet
-		(at 140.97 83.82)
-		(size 19.05 20.32)
-		(exclude_from_sim no)
-		(in_bom yes)
-		(on_board yes)
-		(dnp no)
-		(fields_autoplaced yes)
-		(stroke
-			(width 0.1524)
-			(type solid)
-		)
-		(fill
-			(color 0 0 0 0.0000)
-		)
-		(property "Sheetname" "IO"
-			(at 140.97 83.1084 0)
-			(effects
-				(font
-					(size 1.27 1.27)
-				)
-				(justify left bottom)
-			)
-		)
-		(property "Sheetfile" "io.kicad_sch"
-			(at 140.97 104.7246 0)
-			(effects
-				(font
-					(size 1.27 1.27)
-				)
-				(justify left top)
-			)
-		)
-		(instances
-			(project "ThingsGate-1"
-				(path "/b470e014-149b-42d2-980c-a8a1f9690894"
-					(page "5")
-				)
-			)
