File: Hardware/ThingsGate-1/Modules.kicad_sch (KiCad schematic)
At the start: 5 parts, among them SW1 DSHP03TS-S, U1 CH334R, U2 ThingsCore-1, U7 mPCIE-52P-SLOT, U8 mPCIE-52P-SLOT

Commit message: schematic
Parts:
- added J5: USB_A_Stacked, ThingsGate-1:DUAL_USB-TYPE_A, symbol ThingsGate-1:USB_A_Stacked
- added J7: USB_A, ThingsGate-1:USB_TYPE_A, symbol ThingsGate-1:USB_A
- added U15: TF-123B-ARP9H17, ThingsGate-1:TF-SMD_TF-123-ARP9H15, symbol ThingsGate-1:TF-123B-ARP9H17
- added U6: TCA9535PWR, Package_SO:SSOP-24_5.3x8.2mm_P0.65mm, symbol Interface_Expansion:TCA9535PWR
Other:
- note added: "SPI SD SLOT"
- note added: "USB PORTS"

Commit message: harvester schematic ready
Other:
- note added: "GPIO EXPANDER"
- moved on the sheet: U6, U7, U8
Changed lines of the file:
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@@
 	(rectangle
 		(start 21.844 149.098)
-		(end 160.02 268.478)
+		(end 116.84 268.478)
 		(stroke
 			(width 1.016)
@@
 	)
 	(rectangle
-		(start 168.402 148.844)
-		(end 290.83 267.97)
+		(start 130.302 148.844)
+		(end 200.66 267.97)
 		(stroke
 			(width 1.016)
@@
 	)
 	(rectangle
+		(start 209.55 149.86)
+		(end 294.64 267.97)
+		(stroke
+			(width 1.016)
+			(type dash)
+			(color 132 0 0 1)
+		)
+		(fill
+			(type none)
+		)
+	)
+	(rectangle
 		(start 302.26 139.7)
 		(end 398.78 246.38)
@@
 		(fill
 			(type none)
+		)
+	)
+	(text "GPIO EXPANDER\n"
+		(exclude_from_sim no)
+		(at 237.236 145.288 0)
+		(effects
+			(font
+				(size 5.08 5.08)
+				(thickness 1.016)
+				(bold yes)
+				(color 0 0 255 1)
+			)
 		)
 	)
@@
 	(text "LORAWAN GW SOM"
 		(exclude_from_sim no)
-		(at 202.692 145.034 0)
+		(at 164.592 145.034 0)
 		(effects
 			(font
@@
 	(symbol
 		(lib_id "ThingsGate-1:mPCIE-52P-SLOT")
-		(at 85.09 243.84 0)
+		(at 64.77 245.11 0)
 		(unit 1)
 		(exclude_from_sim no)
@@
 		(fields_autoplaced yes)
 		(property "Reference" "U7"
-			(at 85.09 168.91 0)
+			(at 64.77 170.18 0)
 			(effects
 				(font
@@
 		)
 		(property "Value" "mPCIE-52P-SLOT"
-			(at 85.09 171.45 0)
+			(at 64.77 172.72 0)
 			(effects
 				(font
@@
 		)
 		(property "Footprint" "ThingsGate-1:mpcie-slot_full"
-			(at 86.36 250.698 0)
+			(at 66.04 251.968 0)
 			(effects
 				(font
@@
 		)
 		(property "Datasheet" ""
-			(at 85.09 243.84 0)
+			(at 64.77 245.11 0)
 			(effects
 				(font
@@
 		)
 		(property "Description" ""
-			(at 85.09 243.84 0)
+			(at 64.77 245.11 0)
 			(effects
 				(font
@@
 	(symbol
 		(lib_id "Interface_Expansion:TCA9535PWR")
-		(at 431.8 185.42 0)
+		(at 251.46 200.66 0)
 		(unit 1)
 		(exclude_from_sim no)
@@
 		(fields_autoplaced yes)
 		(property "Reference" "U6"
-			(at 433.9433 157.48 0)
+			(at 253.6033 172.72 0)
 			(effects
 				(font
@@
 		)
 		(property "Value" "TCA9535PWR"
-			(at 433.9433 160.02 0)
+			(at 253.6033 175.26 0)
 			(effects
 				(font
@@
 		)
 		(property "Footprint" "Package_SO:SSOP-24_5.3x8.2mm_P0.65mm"
-			(at 458.47 210.82 0)
+			(at 278.13 226.06 0)
 			(effects
 				(font
@@
 		)
 		(property "Datasheet" "http://www.ti.com/lit/ds/symlink/tca9535.pdf"
-			(at 419.1 162.56 0)
+			(at 238.76 177.8 0)
 			(effects
 				(font
@@
 		)
 		(property "Description" "16-bit I/O expander, I2C and SMBus interface, interrupts, w/o pull-ups, TSSOP-24 package"
-			(at 431.8 185.42 0)
+			(at 251.46 200.66 0)
 			(effects
 				(font
@@
 	(symbol
 		(lib_id "ThingsGate-1:mPCIE-52P-SLOT")
-		(at 220.98 242.57 0)
+		(at 163.83 242.57 0)
 		(unit 1)
 		(exclude_from_sim no)
@@
 		(fields_autoplaced yes)
 		(property "Reference" "U8"
-			(at 220.98 167.64 0)
+			(at 163.83 167.64 0)
 			(effects
 				(font
@@
 		)
 		(property "Value" "mPCIE-52P-SLOT"
-			(at 220.98 170.18 0)
+			(at 163.83 170.18 0)
 			(effects
 				(font
@@
 		)
 		(property "Footprint" "ThingsGate-1:mpcie-slot_full"
-			(at 222.25 249.428 0)
+			(at 165.1 249.428 0)
 			(effects
 				(font
@@
 		)
 		(property "Datasheet" ""
-			(at 220.98 242.57 0)
+			(at 163.83 242.57 0)
 			(effects
 				(font
@@
 		)
 		(property "Description" ""
-			(at 220.98 242.57 0)
-			(effects
-				(font
+			(at 163.83 242.57 0)
+			(effects
+				(font

Commit message: mpcie wire-up
Parts:
- added BT1: S8411-45R, ThingsGate-1:Battery_Holder_CR1220_S8411-45R, symbol Device:Battery_Cell
- added C45, C49, C52: 100n, Capacitor_SMD:C_0603_1608Metric, symbol Device:C
- added C46, C47, C48: 22u, Capacitor_SMD:C_0805_2012Metric, symbol Device:C
- added C50, C53: 1u, Fuse:Fuse_0805_2012Metric, symbol Device:C
- added C51: 10u, Fuse:Fuse_0805_2012Metric, symbol Device:C
- added D12: RED, LED_SMD:LED_0603_1608Metric, symbol Device:LED
- added F5, F6, F7: 500mA, Fuse:Fuse_1206_3216Metric, symbol Device:Fuse
- added J1: Conn_02x07_Odd_Even, Connector_PinHeader_2.54mm:PinHeader_2x07_P2.54mm_Vertical, symbol Connector_Generic:Conn_02x07_Odd_Even
- added R30, R41, R42, R43, R44, R45, R46, R47, R48, R49, R50, R51: 10k, Resistor_SMD:R_0603_1608Metric, symbol Device:R
- added Y1: X322524MSB4SI, Crystal:Crystal_SMD_3225-4Pin_3.2x2.5mm, symbol Device:Crystal_GND24
Connections:
- net GND: now reaches SW1.1
- net GND: now also J5.4 (GND1), J5.8 (GND2), J5.9 (Shield), J7.4 (GND), J7.5 (Shield), SW1.2, SW1.3, U1.14 (GND), U15.10 (SHLD), U15.11 (SHLD), U15.12 (SHLD), U15.13 (SHLD), U15.6 (VSS), U2.2 (GND), U2.30 (GND), U2.4 (GND), U2.41 (GND), U2.47 (GND), U2.6 (GND), U2.S1, U2.S2, U2.S3, U2.S4, U6.12 (GND), U6.2 (A1), U6.21 (A0), U6.3 (A2), U7.15, U7.18, U7.21, U7.26, U7.27, U7.29, U7.34, U7.35, U7.37, U7.4, U7.40, U7.43, U7.50, U7.9, U7.S1, U7.S2, U7.S3, U7.S4, U8.15, U8.18, U8.21, U8.26, U8.27, U8.29, U8.34, U8.35, U8.37, U8.4, U8.40, U8.43, U8.50, U8.9, U8.S1, U8.S2, U8.S3, U8.S4, BT1.2 (-), C45.2, C46.2, C47.2, C48.2, C49.2, C50.1, C51.2, C52.2, C53.2, D12.1 (K), J1.5 (Pin_5), J1.7 (Pin_7), R45.1, R46.1, R48.1, R51.1, Y1.2, Y1.4
- net BOOT2: now reaches SW1.4
- net BOOT2: now also U2.50 (BOOT2), R42.2
- net BOOT1: now reaches SW1.5
- net BOOT1: now also U2.48 (BOOT1), R41.2
- net BOOT0: now reaches SW1.6
- net BOOT0: now also U2.46 (BOOT0), R30.2
- net USB_P1-: now reaches U1.1 (DM4-)
- net USB_P1-: now also J5.2 (D1-)
- net USB1_H-: now reaches U1.10 (DMU-)
- net USB1_H-: now also U2.51 (USB1_N)
- net USB1_H+: now reaches U1.11 (DPU+)
- net USB1_H+: now also U2.49 (USB1_P)
- net 5V: now reaches U1.12 (V5)
- net 5V: now also U2.10 (5VIN), U2.12 (5VIN), U2.8 (5VIN), C46.1, C47.1, C48.1, C50.2, F5.1, F6.1, F7.1
- net HUB_VDD33: now reaches U1.13 (VDD33)
- net HUB_VDD33: now also C49.1, C51.1
- net HUB_XO: now reaches U1.15 (XO)
- net HUB_XO: now also Y1.3
- net HUB_XI: now reaches U1.16 (XI)
- net HUB_XI: now also Y1.1
- net USB_P1+: now reaches U1.2 (DP4+)
- net USB_P1+: now also J5.3 (D1+)
- net USB_P2-: now reaches U1.3 (DM3-)
- net USB_P2-: now also J5.6 (D2-)
- net USB_P2+: now reaches U1.4 (DP3+)
- net USB_P2+: now also J5.7 (D2+)
- net LWUSB_D-: now reaches U1.5 (DM2-)
- net LWUSB_D-: now also U8.36
- net LWUSB_D+: now reaches U1.6 (DP2+)
- net LWUSB_D+: now also U8.38
- net LTE_USB_D-: now reaches U1.7 (DM1-)
- net LTE_USB_D-: now also U7.36
- net LTE_USB_D+: now reaches U1.8 (DP1+)
- net LTE_USB_D+: now also U7.38
- net ETH_LED2: now reaches U2.1 (ETH_LED2)
- net ETH_TXN: now reaches U2.11 (ETH_TXN)
- net UART4_RX: now reaches U2.13 (UART4_RX)
- net UART4_RX: now also J1.13 (Pin_13)
- net I2C1_SDA: now reaches U2.15 (I2C1_SDA)
- net I2C1_SDA: now also U6.23 (SDA), U7.32, U8.32, R43.2
- net SPI4_MISO: now reaches U2.16 (SPI4_MISO)
- net SPI4_MISO: now also U15.7 (SDO/DAT0), U8.49
- net SPI4_SCK: now reaches U2.17 (SPI4_SCK)
- net SPI4_SCK: now also U15.5 (CLK), U8.45
- net CS_AMP_LP: now reaches U2.18 (ADC2_IN3)
- net SPI4_MOSI: now reaches U2.19 (SPI4_MOSI)
- net SPI4_MOSI: now also U15.3 (SDI/CMD), U8.47
- net BUS_VSENSE_LP: now reaches U2.20 (ADC1_IN6)
- net BAT_VSENSE_LP: now reaches U2.22 (ADC2_IN0)
- net UART4_TX: now reaches U2.25 (UART4_TX)
- net UART4_TX: now also J1.14 (Pin_14)
- net I2C1_SCL: now reaches U2.27 (I2C1_SCL)
- net I2C1_SCL: now also U6.22 (SCL), U7.30, U8.30, R44.2
- net IO_EXP_~{INT}: now reaches U2.29 (FDCAN1_RX)
- net IO_EXP_~{INT}: now also U6.1 (~{INT}), R47.1
- net ETH_LED1: now reaches U2.3 (ETH_LED1)
- net SX1301_CSN: now reaches U2.31 (FDCAN1_TX)
- net SX1301_CSN: now also U8.51
- net VBAT_SOM: now reaches U2.32 (VBAT)
- net VBAT_SOM: now also BT1.1 (+)
- net SOM_JTCK: now reaches U2.34 (DBG_JTCK)
- net SOM_JTCK: now also J1.6 (Pin_6)
- net SOM_JTDI: now reaches U2.36 (DBG_JTDI)
- net SOM_JTDI: now also J1.10 (Pin_10)
- net SOM_JTDO: now reaches U2.38 (DBG_JTDO)
- net SOM_JTDO: now also J1.8 (Pin_8)
- net SOM_JTMS: now reaches U2.40 (DBG_JTMS)
- net SOM_JTMS: now also J1.4 (Pin_4)
- net 3V3_SOM: now reaches U2.42 (+3V3_OUT)
- net 3V3_SOM: now also J1.3 (Pin_3)
- net USB2_OTG+: now reaches U2.43 (USB2_P)
- net USB2_OTG+: now also J7.3 (D+)
- net USB2_OTG-: now reaches U2.45 (USB2_N)
- net USB2_OTG-: now also J7.2 (D-)
- net ETH_RXP: now reaches U2.5 (ETH_RXP)
- net SOM_NRST: now reaches U2.52 (NRST)
- net SOM_NRST: now also J1.12 (Pin_12)
- net ETH_RXN: now reaches U2.7 (ETH_RXN)
- net ETH_TXP: now reaches U2.9 (ETH_TXP)
- net SD_CS: now reaches U15.2 (CD/DAT3)
- net SD_CS: now also R50.1
- net 3V3: now reaches U15.4 (VDD)
- net 3V3: now also U6.24 (VCC), U7.2, U7.39, U7.41, U7.52, U8.2, U8.24, U8.39, U8.41, U8.52, C45.1, C52.1, C53.1, R30.1, R41.1, R42.1, R43.1, R44.1, R47.2, R50.2
- net SD_DET: now reaches U15.9 (CD)
- net SD_DET: now also U6.7 (P03), R51.2
- net USB_VB1: now reaches J5.1 (VBUS1)
- net USB_VB1: now also F5.2
- net USB_VB2: now reaches J5.5 (VBUS2)
- net USB_VB2: now also F6.2
- net USIM_DATA: now reaches U7.10
- net USIM_CLK: now reaches U7.12
- net USIM_RST: now reaches U7.14
- net LTE_RST: now reaches U7.22
- net LTE_RST: now also U6.8 (P04), R48.2
- net LED_WWAN: now reaches U7.42
- net LED_WWAN: now also R49.2
- net USIM_DET: now reaches U7.44
- net USIM_VDD: now reaches U7.8
- net MCU_NRST: now reaches U6.10 (P06)
- net MCU_NRST: now also U8.13
- net HARV_STAT1: now reaches U6.4 (P00)
- net HARV_STAT2: now reaches U6.5 (P01)
- net LW_RST: now reaches U6.6 (P02)
- net LW_RST: now also U8.22, R46.2
- net SX1261_NRST: now reaches U6.9 (P05)
- net SX1261_NRST: now also U8.11
- net USB_OTG_VB1: now reaches J7.1 (VBUS)
- net USB_OTG_VB1: now also F7.2
- new net GND_DET: J1.11 (Pin_11), R45.2
- new net WAN_LD: D12.2 (A), R49.1
- no-connect marks 0 -> 59
Other:
- note added: "LW_SPI_MISO"
- note added: "LW_SPI_MOSI"
- moved on the sheet: J5, J7, SW1, U15, U2, U6, U7

Commit message: placement ok
Parts:
- added C54: 100n, Capacitor_SMD:C_0603_1608Metric, symbol Device:C
- added C55, C56, C57: 39p, Capacitor_SMD:C_0603_1608Metric, symbol Device:C
- added R52: 10k, Resistor_SMD:R_0603_1608Metric, symbol Device:R
- added R53, R54: 0R, Resistor_SMD:R_0603_1608Metric, symbol Device:R
- added U16: SMN-305-ARP7, ThingsGate-1:NANO-SIM-SMD_SMN-305-ARP7, symbol ThingsGate-1:SMN-305-ARP7
- J1: footprint Connector_PinHeader_2.54mm:PinHeader_2x07_P2.54mm_Vertical -> Connector_IDC:IDC-Header_2x07_P2.54mm_Vertical
- J7: footprint ThingsGate-1:USB_TYPE_A -> ThingsGate-1:USB-A-TH_AF-ZJB13.7
- R45: value 10k -> 100R
- Y1: value X322524MSB4SI -> X322512MOB4SI
Connections:
- net GND: now also C54.1, C55.2, C56.2, C57.2, U16.10 (GND), U16.11 (GND), U16.5 (GND), U16.9 (GND)
- net USIM_CLK: now also C56.1, U16.3 (CLK)
- net USIM_DATA: now also C57.1, R52.1, U16.7 (I/O)
- net USIM_DET: now also U16.8 (SW)
- net USIM_RST: now also C55.1, U16.2 (RST)
- net USIM_VDD: now also C54.2, R52.2, U16.1 (VCC)
- net at U7.11: now also R53.1
- net at U7.13: now also R54.2
- net SX1261_NRST_LTE: now reaches U6.11 (P07)
- net SX1261_NRST_LTE: now also R53.2
- net MCU_NRST_LTE: now reaches U6.13 (P10)
- net MCU_NRST_LTE: now also R54.1
- no-connect marks 59 -> 68
Other:
- moved on the sheet: C46, C47, C48, C49, C50, C51, C52, C53, F5, F7, J5, J7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

Commit message: layout finished. checks and fab files remaining
Connections:
- net BOOT0: now also SW1.4; no longer SW1.6
- net BOOT2: now also SW1.6; no longer SW1.4
- net GND: no longer J5.9 (Shield), J7.5 (Shield)
- net HARV_STAT1: now also U6.6 (P02); no longer U6.4 (P00)
- net LTE_RST: now also U6.7 (P03); no longer U6.8 (P04)
- net LW_RST: now also U6.9 (P05); no longer U6.6 (P02)
- net MCU_NRST_LTE: now also U6.14 (P11); no longer U6.13 (P10)
- net SD_DET: now also U6.8 (P04); no longer U6.7 (P03)
- net SX1261_NRST: now also U6.11 (P07); no longer U6.9 (P05)
- net SX1261_NRST_LTE: now also U6.13 (P10); no longer U6.11 (P07)
- new net CHASSIS: J5.9 (Shield), J7.5 (Shield)
- no-connect marks 68 -> 67
Other:
- moved on the sheet: SW1

Commit message: final fab files and checks done
Parts:
- added TP7, TP8: TestPoint, TestPoint:TestPoint_Pad_D1.5mm, symbol Connector:TestPoint
Connections:
- net SOM_NRST: now also TP8.1
- net PWR_ONRST: now reaches U2.44 (PWR_ONRST)
- net PWR_ONRST: now also TP7.1
Changed lines of the file:
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@@
 	)
 	(junction
+		(at 86.36 107.95)
+		(diameter 0)
+		(color 0 0 0 0)
+	)
+	(junction
 		(at 87.63 259.08)
 		(diameter 0)
@@
 	)
 	(no_connect
+		(at 267.97 187.96)
+	)
+	(no_connect
 		(at 78.74 220.98)
 	)
@@
 	)
 	(no_connect
-		(at 82.55 97.79)
-	)
-	(no_connect
 		(at 118.11 39.37)
 	)
@@
 	(wire
 		(pts
+			(xy 82.55 97.79) (xy 100.33 97.79)
+		)
+		(stroke
+			(width 0)
+			(type default)
+		)
+	)
+	(wire
+		(pts
 			(xy 231.14 228.6) (xy 232.41 228.6)
 		)
@@
 	(wire
 		(pts
+			(xy 184.15 203.2) (xy 199.39 203.2)
+		)
+		(stroke
+			(width 0)
+			(type default)
+		)
+	)
+	(wire
+		(pts
 			(xy 54.61 205.74) (xy 55.88 205.74)
 		)
@@
 	(wire
 		(pts
+			(xy 86.36 107.95) (xy 92.71 107.95)
+		)
+		(stroke
+			(width 0)
+			(type default)
+		)
+	)
+	(wire
+		(pts
 			(xy 91.44 64.77) (xy 82.55 64.77)
 		)
@@
 	(wire
 		(pts
-			(xy 307.34 172.72) (xy 307.34 170.18)
-		)
-		(stroke
-			(width 0)
-			(type default)
-		)
-	)
-	(wire
-		(pts
 			(xy 318.77 48.26) (xy 318.77 45.72)
 		)
@@
 	(wire
 		(pts
+			(xy 86.36 110.49) (xy 86.36 107.95)
+		)
+		(stroke
+			(width 0)
+			(type default)
+		)
+	)
+	(wire
+		(pts
 			(xy 30.48 82.55) (xy 44.45 82.55)
 		)
@@
 	(wire
 		(pts
-			(xy 82.55 107.95) (xy 92.71 107.95)
+			(xy 82.55 107.95) (xy 86.36 107.95)
 		)
 		(stroke
@@
 	(wire
 		(pts
-			(xy 184.15 203.2) (xy 199.39 203.2)
-		)
-		(stroke
-			(width 0)
-			(type default)
-		)
-	)
-	(wire
-		(pts
 			(xy 66.04 231.14) (xy 63.5 231.14)
 		)
@@
 		)
 	)
+	(label "PWR_ONRST"
+		(at 100.33 97.79 180)
+		(effects
+			(font
+				(size 1.27 1.27)
+			)
+			(justify right bottom)
+		)
+	)
 	(label "SOM_NRST"
 		(at 140.97 52.07 180)
@@
 	(symbol
 		(lib_id "power:GND")
-		(at 307.34 170.18 270)
+		(at 307.34 172.72 270)
 		(mirror x)
 		(unit 1)
@@
 		(fields_autoplaced yes)
 		(property "Reference" "#PWR0135"
-			(at 300.99 170.18 0)
+			(at 300.99 172.72 0)
 			(effects
 				(font
@@
 		)
 		(property "Value" "GND"
-			(at 302.26 170.18 0)
+			(at 302.26 172.72 0)
 			(effects
 				(font
@@
 		)
 		(property "Footprint" ""
-			(at 307.34 170.18 0)
+			(at 307.34 172.72 0)
 			(effects
 				(font
@@
 		)
 		(property "Datasheet" ""
-			(at 307.34 170.18 0)
+			(at 307.34 172.72 0)
 			(effects
 				(font
@@
 		)
 		(property "Description" "Power symbol creates a global label with name \"GND\" , ground"
-			(at 307.34 170.18 0)
+			(at 307.34 172.72 0)
 			(effects
 				(font
@@
 	)
 	(symbol
+		(lib_id "Connector:TestPoint")
+		(at 100.33 97.79 270)
+		(unit 1)
+		(exclude_from_sim no)
+		(in_bom yes)
+		(on_board yes)
+		(dnp no)
+		(fields_autoplaced yes)
+		(property "Reference" "TP7"
+			(at 105.41 96.5199 90)
+			(effects
+				(font
+					(size 1.27 1.27)
+				)
+				(justify left)
+			)
+		)
+		(property "Value" "TestPoint"
+			(at 105.41 99.0599 90)
+			(effects
+				(font
+					(size 1.27 1.27)
+				)
+				(justify left)
+			)
+		)
+		(property "Footprint" "TestPoint:TestPoint_Pad_D1.5mm"
+			(at 100.33 102.87 0)
+			(effects
+				(font
+					(size 1.27 1.27)
+				)
+				(hide yes)
+			)
+		)
+		(property "Datasheet" "~"
+			(at 100.33 102.87 0)
+			(effects
+				(font
+					(size 1.27 1.27)
+				)
+				(hide yes)
+			)
+		)
+		(property "Description" "test point"
+			(at 100.33 97.79 0)
+			(effects
+				(font
+					(size 1.27 1.27)
+				)
+				(hide yes)
+			)
+		)
+		(pin "1"
+		)
+		(instances
+			(project "ThingsGate-1"
+				(path "/b470e014-149b-42d2-980c-a8a1f9690894/e00fcd44-9245-479e-a548-7d5d1555425b"
+					(reference "TP7")
+					(unit 1)
+				)
+			)
+		)
+	)
+	(symbol
 		(lib_id "power:GND")
 		(at 198.12 205.74 90)
@@
 					(unit 1)
 				)
+			)
+		)
+	)
+	(symbol
+		(lib_id "Connector:TestPoint")
+		(at 86.36 110.49 180)
+		(unit 1)
+		(exclude_from_sim no)
+		(in_bom yes)
+		(on_board yes)
+		(dnp no)
+		(fields_autoplaced yes)
+		(property "Reference" "TP8"
+			(at 88.9 112.5219 0)
+			(effects
+				(font
+					(size 1.27 1.27)
+				)
+				(justify right)
+			)
+		)
+		(property "Value" "TestPoint"
+			(at 88.9 115.0619 0)
+			(effects
+				(font
+					(size 1.27 1.27)
+				)
+				(justify right)
+			)
+		)
+		(property "Footprint" "TestPoint:TestPoint_Pad_D1.5mm"
+			(at 81.28 110.49 0)
+			(effects
+				(font
+					(size 1.27 1.27)
+				)
+				(hide yes)
+			)
+		)
+		(property "Datasheet" "~"
+			(at 81.28 110.49 0)
+			(effects
+				(font
+					(size 1.27 1.27)
+				)
+				(hide yes)
+			)
+		)
+		(property "Description" "test point"
+			(at 86.36 110.49 0)
+			(effects
+				(font
+					(size 1.27 1.27)
+				)
+				(hide yes)
+			)
+		)
+		(pin "1"
+		)
+		(instances
+			(project "ThingsGate-1"
+				(path "/b470e014-149b-42d2-980c-a8a1f9690894/e00fcd44-9245-479e-a548-7d5d1555425b"
+					(reference "TP8")
+					(unit 1)
+				)
