File: Hardware/ThingsGate-1/Power.kicad_sch (KiCad schematic)
At the start: 20 parts, among them Q1 Si4435DDY, Q2 Si4435DDY, Q3 Si4435DDY, T1 H1102NL, U10 TPS54331DR, U11 RJ45-202-007-02, U3 POE_PD_Module, U9 TPS54331DR

Commit message: schematic
Parts:
- removed D3, D5: BZT52C10, Diode_SMD:D_SOD-123, symbol Device:D_Zener
- removed Q2: Si4435DDY, ThingsGate-1:SO-8_3.9x4.9mm_P1.27mm, symbol ThingsGate-1:Si4435DDY
- added C1, C13, C2, C20, C21, C24, C25, C26, C3, C4, C5, C6: 100n, Capacitor_SMD:C_0603_1608Metric, symbol Device:C
- added C10, C9: 330uF 50V, Capacitor_SMD:CP_Elec_10x10.5, symbol Device:C_Polarized
- added C11, C12: 10u, Capacitor_SMD:C_0805_2012Metric, symbol Device:C
- added C14, C15: 47u, Capacitor_SMD:C_0805_2012Metric, symbol Device:C
- added C16, C7: 1n, Capacitor_SMD:C_0603_1608Metric, symbol Device:C
- added C17: 47p, Capacitor_SMD:C_0603_1608Metric, symbol Device:C
- added C18, C19, C22, C23: 4.7u, Capacitor_SMD:C_0805_2012Metric, symbol Device:C
- added C27: 4.7n, Capacitor_SMD:C_0603_1608Metric, symbol Device:C
- added C28: 39p, Capacitor_SMD:C_0603_1608Metric, symbol Device:C
- added C29, C30: 22u, Capacitor_SMD:C_0805_2012Metric, symbol Device:C
- added C8: 10u, Fuse:Fuse_0805_2012Metric, symbol Device:C
- added D3, D5, D7: SMAJ15CA, Diode_SMD:D_SMA, symbol Diode:SMAJ15CA
- added D6: BZT52C10, Diode_SMD:D_SOD-123, symbol Device:D_Zener
- added F1, F2, F3, F4: 4A, Fuse:Fuse_1206_3216Metric, symbol Device:Fuse
- added J3, J4, J6: 691313710002, ThingsGate-1:691313710002, symbol ThingsGate-1:691313710002
- added L4: 2.2u, ThingsCore-1:L_0805_2016, symbol Device:L
- added Q2, Q4, Q5: Si4178DY, ThingsGate-1:SO-8_3.9x4.9mm_P1.27mm, symbol ThingsGate-1:Si4178DY
- added R10: 3.24k, Resistor_SMD:R_0603_1608Metric, symbol Device:R
- added R11: 29.4k, Resistor_SMD:R_0603_1608Metric, symbol Device:R
- added R12, R14: 332k, Resistor_SMD:R_0603_1608Metric, symbol Device:R
- added R13, R15: 68.1k, Resistor_SMD:R_0603_1608Metric, symbol Device:R
- added R16: 49.4k, Resistor_SMD:R_0603_1608Metric, symbol Device:R
- added R17, R7, R8, R9: 10k, Resistor_SMD:R_0603_1608Metric, symbol Device:R
- added R18: 1.91k, Resistor_SMD:R_0603_1608Metric, symbol Device:R
- added R2: 100K, Resistor_SMD:R_0603_1608Metric, symbol Device:R
- added R3, R4, R5, R6: 75R, Resistor_SMD:R_0603_1608Metric, symbol Device:R
- added U12, U13, U4: LM74700, Package_TO_SOT_SMD:SOT-23-6, symbol Power_Management:LM74700
- R1: value R -> 100K
Connections:
- net VSOL_G: now reaches R1.1
- net VSOL_G: now also D4.2 (A), Q3.4 (G)
- net GND: now reaches R1.2
- net GND: now also D1.2 (A), D2.2 (A), U10.7 (GND), U10.9 (EP), U11.10 (-), U11.12 (-), U3.7 (-VDC), U9.7 (GND), U9.9 (EP), C1.2, C10.2, C11.2, C12.2, C14.2, C15.2, C17.2, C18.2, C19.2, C20.2, C21.2, C22.2, C23.2, C24.2, C26.2, C28.2, C29.2, C3.2, C30.2, C5.2, C8.2, C9.2, D3.1 (A1), D5.1 (A1), D7.1 (A1), J3.1, J4.1, J6.1, R10.2, R11.2, R13.2, R15.2, R16.2, R18.2, R2.2, U12.2 (GND), U13.2 (GND), U4.2 (GND)
- net VA1: now reaches U3.1 (VA1)
- net VA1: now also T1.15 (CT4), R5.1
- net VA2: now reaches U3.2 (VA2)
- net VA2: now also T1.10 (CT3), R3.1
- net VB1: now reaches U3.3 (VB1)
- net VB1: now also U11.4, U11.5, R4.1
- net VB2: now reaches U3.4 (VB2)
- net VB2: now also U11.7, U11.8, R6.1
- net VDC_POE: now reaches U3.8 (+VDC)
- net VDC_POE: now also C9.1, L4.1
- net VSOL: now reaches D4.1 (K)
- net VSOL: now also Q3.1 (S), Q3.2 (S), Q3.3 (S)
- net VSOL_CONN: now reaches Q3.5 (D), Q3.6 (D), Q3.7 (D), Q3.8 (D)
- net VSOL_CONN: now also J4.2
- net 3V3_BOOT: now reaches U9.1 (BOOT)
- net 3V3_BOOT: now also C13.2
- net VBUS: now reaches U9.2 (VIN)
- net VBUS: now also U10.2 (VIN), C18.1, C19.1, C20.1, C22.1, C23.1, C24.1, F3.2, R12.1, R14.1
- net 3V3_EN: now reaches U9.3 (EN)
- net 3V3_EN: now also R12.2, R13.1
- net 3V3_SS: now reaches U9.4 (SS)
- net 3V3_SS: now also C21.1
- net 3V3_VS: now reaches U9.5 (VSENSE)
- net 3V3_VS: now also R10.1, R9.2
- net 3V3_C: now reaches U9.6 (COMP)
- net 3V3_C: now also C16.1, C17.1
- net 3V3_PH: now reaches U9.8 (PH)
- net 3V3_PH: now also D2.1 (K), L1.1, C13.1
- net 12VBAT_HARV: now reaches Q1.1 (S), Q1.2 (S), Q1.3 (S)
- net 12VBAT_HARV: now also D6.1 (K)
- net VBAT_G: now reaches Q1.4 (G)
- net VBAT_G: now also D6.2 (A), R2.1
- net 12VBAT: now reaches Q1.5 (D), Q1.6 (D), Q1.7 (D), Q1.8 (D)
- net 12VBAT: now also C1.1, C2.1, D3.2 (A2), F2.2, Q2.1 (S), Q2.2 (S), Q2.3 (S), U4.3 (EN), U4.6 (ANODE)
- net 5V_PH: now reaches D1.1 (K)
- net 5V_PH: now also L2.1, U10.8 (PH), C25.1
- net 5V_BOOT: now reaches U10.1 (BOOT)
- net 5V_BOOT: now also C25.2
- net 5V_EN: now reaches U10.3 (EN)
- net 5V_EN: now also R14.2, R15.1
- net 5V_SS: now reaches U10.4 (SS)
- net 5V_SS: now also C26.1
- net 5V_VS: now reaches U10.5 (VSENSE)
- net 5V_VS: now also R17.2, R18.1
- net 5V_C: now reaches U10.6 (COMP)
- net 5V_C: now also C27.1, C28.1
- net RX+: now reaches T1.11 (RX+)
- net RX+: now also U11.3 (RX+)
- net TX-: now reaches T1.14 (TX-)
- net TX-: now also U11.2 (TX-)
- net TX+: now reaches T1.16 (TX+)
- net TX+: now also U11.1 (TX+)
- net RX-: now reaches T1.9 (RX-)
- net RX-: now also U11.6 (RX-)
- net 5V: now reaches L2.2
- net 5V: now also C29.1, C30.1, R17.1
- net 3V3: now reaches L1.2
- net 3V3: now also C14.1, C15.1, R9.1
- net ETH_LED_1: now reaches U11.11 (+)
- net ETH_LED_1: now also R8.2
- net CHASSIS: now reaches U11.13 (SHIELD)
- net CHASSIS: now also C7.1
- net ETH_LED_2: now reaches U11.9 (+)
- net ETH_LED_2: now also R7.2
- new net: C7.2, R3.2, R4.2, R5.2, R6.2
- new net: C8.1, F4.1, L4.2
- new net: C27.2, R16.1
- new net: C16.2, R11.1
- new net 12VBAT_CONN: F2.1, J3.2
- new net 12VPOE: C5.1, C6.1, D7.2 (A2), F4.2, Q5.1 (S), Q5.2 (S), Q5.3 (S), U13.3 (EN), U13.6 (ANODE)
- new net 12VPSU: C3.1, C4.1, D5.2 (A2), F1.2, Q4.1 (S), Q4.2 (S), Q4.3 (S), U12.3 (EN), U12.6 (ANODE)
- new net 12VPSU_CONN: F1.1, J6.2
- new net LED1: R8.1
- new net LED2: R7.1
- new net OR1G: Q2.4 (G), U4.5 (GATE)
- new net OR2G: Q4.4 (G), U12.5 (GATE)
- new net OR3G: Q5.4 (G), U13.5 (GATE)
- new net VBUS_FUSE: C10.1, C11.1, C12.1, F3.1, Q2.5 (D), Q2.6 (D), Q2.7 (D), Q2.8 (D), Q4.5 (D), Q4.6 (D), Q4.7 (D), Q4.8 (D), Q5.5 (D), Q5.6 (D), Q5.7 (D), Q5.8 (D), U12.4 (CATHODE), U13.4 (CATHODE), U4.4 (CATHODE)
- new net VCAP_1: C2.2, U4.1 (VCAP)
- new net VCAP_2: C4.2, U12.1 (VCAP)
- new net VCAP_3: C6.2, U13.1 (VCAP)
- no-connect marks 0 -> 8
Other:
- note added: "12V DCIN"
- note added: "POWER ORING"
- note added: "SOLAR PANEL"
- note removed: "12VIN JACK"
- moved on the sheet: D2, D4, H1, H2, H3, H4, L1, Q3, T1, U11, U3, U9

Commit message: harvester schematic ready
Parts:
- added C39, C40, C41, C42: 100n, Capacitor_SMD:C_0603_1608Metric, symbol Device:C
- added D10, D11, D9: 1N5817WS, Diode_SMD:D_SOD-323, symbol Diode:1N4148WS
- added R31: 0.015R, Resistor_SMD:R_1206_3216Metric, symbol Device:R
- added R32, R34, R35, R36, R38, R40: 100K, Resistor_SMD:R_0603_1608Metric, symbol Device:R
- added R33: 5.1K, Resistor_SMD:R_0603_1608Metric, symbol Device:R
- added R37: 10K, Resistor_SMD:R_0603_1608Metric, symbol Device:R
- added R39: 10k, Resistor_SMD:R_0603_1608Metric, symbol Device:R
- added U14: LM324, Package_SO:SOIC-14_3.9x8.7mm_P1.27mm, symbol Amplifier_Operational:LM324
- L4: footprint ThingsCore-1:L_0805_2016 -> ThingsGate-1:L_0805_2016
Connections:
- net 12VBAT_HARV: now also R38.2
- net 3V3: now also D10.1 (K), D11.1 (K), D9.1 (K)
- net 5V: now also C39.1, U14.4 (V+)
- net GND: now also C39.2, C40.1, C41.1, C42.1, R31.2, R37.1, R39.1, U14.11 (V-), U14.2 (-); no longer J4.1
- net VBUS: now also R36.2
- new net BAT_VSENSE: R38.1, R39.2, U14.10 (+)
- new net BAT_VSENSE_LP: C42.2, D11.2 (A), R40.2
- new net BAT_VSENSE_N: R40.1, U14.8, U14.9 (-)
- new net BUS_VSENSE: R36.1, R37.2, U14.5 (+)
- new net BUS_VSENSE_LP: C41.2, D10.2 (A), R35.2
- new net BUS_VSENSE_N: R35.1, U14.6 (-), U14.7
- new net S_AMP_LP: C40.2, D9.2 (A), R32.2
- new net S_AMP_OUT: R32.1, R34.2, U14.1
- new net S_AMP_P: R33.2, R34.1, U14.3 (+)
- new net VSOL_SENSE: J4.1, R31.1, R33.1
Other:
- note added: "POWER SENSORS"
- moved on the sheet: C1, C10, C11, C12, C13, C14, C15, C16, C17, C18, C19, C2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

Commit message: mpcie wire-up
Parts:
- added C43, C44: 100n, Capacitor_SMD:C_0603_1608Metric, symbol Device:C
- U3: Part (none) -> SDAPO DP9700
Connections:
- net GND: now also C43.2, C44.2
- net ETH_TXP: now reaches T1.1 (TD+)
- net CT_ETH_PHY: now reaches T1.2 (CT1)
- net CT_ETH_PHY: now also T1.7 (CT2), C43.1, C44.1
- net ETH_TXN: now reaches T1.3 (TD-)
- net ETH_RXP: now reaches T1.6 (RD+)
- net ETH_RXN: now reaches T1.8 (RD-)
- net LED1 renamed ETH_LED1
- net LED2 renamed ETH_LED2
- net S_AMP_LP renamed CS_AMP_LP

Commit message: placement ok
Connections:
- net GND: now also U14.3 (+); no longer U14.2 (-)
- net S_AMP_P: now also U14.2 (-); no longer U14.3 (+)
- no-connect marks 8 -> 12
Other:
- moved on the sheet: R33, R34

Commit message: layout finished. checks and fab files remaining
Connections:
- net CHASSIS: now also H1.1, H2.1, H3.1, H4.1

Commit message: final fab files and checks done
Parts:
- added TP1, TP2, TP3, TP4, TP5: TestPoint, TestPoint:TestPoint_Pad_D1.5mm, symbol Connector:TestPoint
- C7: footprint Capacitor_SMD:C_0603_1608Metric -> Capacitor_SMD:C_1206_3216Metric
Connections:
- net 12VPOE: now also TP5.1
- net 3V3: now also TP3.1
- net 5V: now also TP4.1
- net VBUS: now also TP1.1
- net VBUS_FUSE: now also TP2.1
Other:
- note added: "EFI 2KV"
