File: Hardware/ThingsGate-1/ThingsGate-1.kicad_pcb (KiCad board)
At the start: 4 copper layers, 100 x 100 mm, 17 parts, among them J1 USB_A_Stacked, J2 USB_A, SW1 DSHP03TS-S, T1 H1102NL, U11 RJ45-202-007-02, U2 ThingsCore-1, U3 POE_PD_Module, U6 TF-123B-ARP9H17, U7 mPCIE-52P-SLOT, U8 mPCIE-52P-SLOT

Commit message: schematic
Parts:
- removed H1, H2, H3, H4: MountingHole_Pad, MountingHole:MountingHole_3.2mm_M3_DIN965_Pad_TopBottom
- removed J1: USB_A_Stacked, ThingsGate-1:DUAL_USB-TYPE_A
- removed J2: USB_A, ThingsGate-1:USB_TYPE_A
- removed REF** (x3): TerminalBlock_Phoenix_MKDS-1,5-2-5.08_1x02_P5.08mm_Horizont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, TerminalBlock_Phoenix:TerminalBlock_Phoenix_MKDS-1,5-2-5.08_1x02_P5.08mm_Horizontal
- removed SW1: DSHP03TS-S, ThingsGate-1:SW-SMD_DSHP03TS-S
- removed T1: H1102NL, ThingsGate-1:H1102NL
- removed U11: RJ45-202-007-02, ThingsGate-1:RJ45-TH_RJ45-202-007-02
- removed U2: ThingsCore-1, ThingsGate-1:ThingsCore-1
- removed U3: POE_PD_Module, ThingsGate-1:SDAPO_DP9700
- removed U6: TF-123B-ARP9H17, ThingsGate-1:TF-SMD_TF-123-ARP9H15
- removed U7, U8: mPCIE-52P-SLOT, ThingsGate-1:mpcie-slot_full

Commit message: harvester schematic ready
Parts:
- added C1: 100n, Capacitor_SMD:C_0603_1608Metric, F.Cu at (145.2, 58.5)
- added C10: 330uF 50V, Capacitor_SMD:CP_Elec_10x10.5, F.Cu at (159.1, 95.4)
- added C11: 10u, Capacitor_SMD:C_0805_2012Metric, F.Cu at (178.3, 78.8)
- added C12: 10u, Capacitor_SMD:C_0805_2012Metric, F.Cu at (178.3, 81.8)
- added C13: 100n, Capacitor_SMD:C_0603_1608Metric, F.Cu at (145.2, 76.0)
- added C14: 47u, Capacitor_SMD:C_0805_2012Metric, F.Cu at (178.3, 84.8)
- added C15: 47u, Capacitor_SMD:C_0805_2012Metric, F.Cu at (178.3, 87.8)
- added C16: 1n, Capacitor_SMD:C_0603_1608Metric, F.Cu at (149.2, 58.5)
- added C17: 47p, Capacitor_SMD:C_0603_1608Metric, F.Cu at (149.2, 61.0)
- added C18: 4.7u, Capacitor_SMD:C_0805_2012Metric, F.Cu at (178.3, 90.8)
- added C19: 4.7u, Capacitor_SMD:C_0805_2012Metric, F.Cu at (182.8, 78.8)
- added C2: 100n, Capacitor_SMD:C_0603_1608Metric, F.Cu at (145.2, 61.0)
- added C20: 100n, Capacitor_SMD:C_0603_1608Metric, F.Cu at (149.2, 63.5)
- added C21: 100n, Capacitor_SMD:C_0603_1608Metric, F.Cu at (149.2, 66.0)
- added C22: 4.7u, Capacitor_SMD:C_0805_2012Metric, F.Cu at (182.8, 81.8)
- added C23: 4.7u, Capacitor_SMD:C_0805_2012Metric, F.Cu at (182.8, 84.8)
- added C24: 100n, Capacitor_SMD:C_0603_1608Metric, F.Cu at (149.2, 68.5)
- added C25: 100n, Capacitor_SMD:C_0603_1608Metric, F.Cu at (149.2, 71.0)
- added C26: 100n, Capacitor_SMD:C_0603_1608Metric, F.Cu at (149.2, 73.5)
- added C27: 4.7n, Capacitor_SMD:C_0603_1608Metric, F.Cu at (149.2, 76.0)
- added C28: 39p, Capacitor_SMD:C_0603_1608Metric, F.Cu at (153.2, 58.5)
- added C29: 22u, Capacitor_SMD:C_0805_2012Metric, F.Cu at (182.8, 87.8)
- added C3: 100n, Capacitor_SMD:C_0603_1608Metric, F.Cu at (145.2, 63.5)
- added C30: 22u, Capacitor_SMD:C_0805_2012Metric, F.Cu at (182.8, 90.8)
- added C31: 10u, Fuse:Fuse_0805_2012Metric, F.Cu at (197.6, 68.7)
- added C32: 100n, Capacitor_SMD:C_0603_1608Metric, F.Cu at (189.0, 58.5)
- added C33: 1u, Fuse:Fuse_0805_2012Metric, F.Cu at (197.6, 71.7)
- added C34: 4.7u, Fuse:Fuse_0805_2012Metric, F.Cu at (197.6, 74.6)
- added C35: 1u, Fuse:Fuse_0805_2012Metric, F.Cu at (197.6, 77.6)
- added C36: 100n, Capacitor_SMD:C_0603_1608Metric, F.Cu at (189.0, 61.0)
- added C37: 1u, Fuse:Fuse_0805_2012Metric, F.Cu at (197.6, 80.5)
- added C38: 100n, Capacitor_SMD:C_0603_1608Metric, F.Cu at (189.0, 63.5)
- added C39: 100n, Capacitor_SMD:C_0603_1608Metric, F.Cu at (153.2, 61.0)
- added C4: 100n, Capacitor_SMD:C_0603_1608Metric, F.Cu at (145.2, 66.0)
- added C40: 100n, Capacitor_SMD:C_0603_1608Metric, F.Cu at (153.2, 63.5)
- added C41: 100n, Capacitor_SMD:C_0603_1608Metric, F.Cu at (153.2, 66.0)
- added C42: 100n, Capacitor_SMD:C_0603_1608Metric, F.Cu at (153.2, 68.5)
- added C5: 100n, Capacitor_SMD:C_0603_1608Metric, F.Cu at (145.2, 68.5)
- added C6: 100n, Capacitor_SMD:C_0603_1608Metric, F.Cu at (145.2, 71.0)
- added C7: 1n, Capacitor_SMD:C_0603_1608Metric, F.Cu at (145.2, 73.5)
- added C8: 10u, Fuse:Fuse_0805_2012Metric, F.Cu at (139.2, 121.6)
- added C9: 330uF 50V, Capacitor_SMD:CP_Elec_10x10.5, F.Cu at (159.1, 83.3)
- added D1: B360, Diode_SMD:D_SMA, F.Cu at (175.0, 103.7)
- added D10: 1N5817WS, Diode_SMD:D_SOD-323, F.Cu at (139.1, 115.7)
- added D11: 1N5817WS, Diode_SMD:D_SOD-323, F.Cu at (139.1, 118.7)
- added D2: B360, Diode_SMD:D_SMA, F.Cu at (175.0, 108.2)
- added D3: SMAJ15CA, Diode_SMD:D_SMA, F.Cu at (175.0, 112.8)
- added D4: BZT52C10, Diode_SMD:D_SOD-123, F.Cu at (181.9, 119.5)
- added D5: SMAJ15CA, Diode_SMD:D_SMA, F.Cu at (175.0, 117.3)
- added D6: BZT52C10, Diode_SMD:D_SOD-123, F.Cu at (181.9, 122.9)
- added D7: SMAJ15CA, Diode_SMD:D_SMA, F.Cu at (175.0, 121.9)
- added D8: 1N5817WS, Diode_SMD:D_SOD-323, F.Cu at (206.8, 58.7)
- added D9: 1N5817WS, Diode_SMD:D_SOD-323, F.Cu at (139.1, 112.8)
- added F1: 4A, Fuse:Fuse_1206_3216Metric, F.Cu at (181.8, 103.0)
- added F2: 4A, Fuse:Fuse_1206_3216Metric, F.Cu at (181.8, 106.3)
- added F3: 4A, Fuse:Fuse_1206_3216Metric, F.Cu at (181.8, 109.6)
- added F4: 4A, Fuse:Fuse_1206_3216Metric, F.Cu at (181.8, 112.9)
- added H1: MountingHole_Pad, MountingHole:MountingHole_3.2mm_M3_DIN965_Pad_TopBottom, F.Cu at (133.4, 101.0)
- added H2: MountingHole_Pad, MountingHole:MountingHole_3.2mm_M3_DIN965_Pad_TopBottom, F.Cu at (133.4, 108.1)
- added H3: MountingHole_Pad, MountingHole:MountingHole_3.2mm_M3_DIN965_Pad_TopBottom, F.Cu at (133.4, 115.3)
- added H4: MountingHole_Pad, MountingHole:MountingHole_3.2mm_M3_DIN965_Pad_TopBottom, F.Cu at (133.4, 122.4)
- added J3: 691313710002, ThingsGate-1:691313710002, F.Cu at (136.5, 59.9)
- added J4: 691313710002, ThingsGate-1:691313710002, F.Cu at (136.5, 73.3)
- added J5: USB_A_Stacked, ThingsGate-1:DUAL_USB-TYPE_A, F.Cu at (127.7, 40.8)
- added J6: 691313710002, ThingsGate-1:691313710002, F.Cu at (136.5, 86.7)
- added J7: USB_A, ThingsGate-1:USB_TYPE_A, F.Cu at (145.5, 44.4)
- added L1: 6.8u, ThingsGate-1:L_0730-6R8M, F.Cu at (171.2, 81.7)
- added L2: 6.8u, ThingsGate-1:L_0730-6R8M, F.Cu at (171.2, 90.6)
- added L3: 6.8u, ThingsGate-1:L_0730-6R8M, F.Cu at (204.8, 71.7)
- added L4: 2.2u, ThingsGate-1:L_0805_2016, F.Cu at (145.1, 122.2)
- added Q1: Si4435DDY, ThingsGate-1:SO-8_3.9x4.9mm_P1.27mm, F.Cu at (147.4, 80.6)
- added Q2: Si4178DY, ThingsGate-1:SO-8_3.9x4.9mm_P1.27mm, F.Cu at (147.4, 87.2)
- added Q3: Si4435DDY, ThingsGate-1:SO-8_3.9x4.9mm_P1.27mm, F.Cu at (147.4, 93.8)
- added Q4: Si4178DY, ThingsGate-1:SO-8_3.9x4.9mm_P1.27mm, F.Cu at (147.4, 100.4)
- added Q5: Si4178DY, ThingsGate-1:SO-8_3.9x4.9mm_P1.27mm, F.Cu at (147.4, 107.0)
- added Q6: Si4178DY, ThingsGate-1:SO-8_3.9x4.9mm_P1.27mm, F.Cu at (191.2, 70.6)
- added Q7: Si4178DY, ThingsGate-1:SO-8_3.9x4.9mm_P1.27mm, F.Cu at (191.2, 77.2)
- added R1: 100K, Resistor_SMD:R_0603_1608Metric, F.Cu at (153.2, 71.0)
- added R10: 3.24k, Resistor_SMD:R_0603_1608Metric, F.Cu at (157.2, 73.5)
- added R11: 29.4k, Resistor_SMD:R_0603_1608Metric, F.Cu at (157.2, 76.0)
- added R12: 332k, Resistor_SMD:R_0603_1608Metric, F.Cu at (161.3, 58.5)
- added R13: 68.1k, Resistor_SMD:R_0603_1608Metric, F.Cu at (161.3, 61.0)
- added R14: 332k, Resistor_SMD:R_0603_1608Metric, F.Cu at (161.3, 63.5)
- added R15: 68.1k, Resistor_SMD:R_0603_1608Metric, F.Cu at (161.3, 66.0)
- added R16: 49.4k, Resistor_SMD:R_0603_1608Metric, F.Cu at (161.3, 68.5)
- added R17: 10k, Resistor_SMD:R_0603_1608Metric, F.Cu at (161.3, 71.0)
- added R18: 1.91k, Resistor_SMD:R_0603_1608Metric, F.Cu at (161.3, 73.5)
- added R19: 10R, Resistor_SMD:R_1206_3216Metric, F.Cu at (201.8, 58.9)
- added R2: 100K, Resistor_SMD:R_0603_1608Metric, F.Cu at (153.2, 73.5)
- added R20: 0.015R, Resistor_SMD:R_1206_3216Metric, F.Cu at (201.8, 62.1)
- added R21: 10k, Resistor_SMD:R_0603_1608Metric, F.Cu at (189.0, 66.0)
- added R22: 10k, Resistor_SMD:R_0603_1608Metric, F.Cu at (193.0, 58.5)
- added R23: 100k, Resistor_SMD:R_0603_1608Metric, F.Cu at (193.0, 61.0)
- added R24: 7.15k, Resistor_SMD:R_0603_1608Metric, F.Cu at (193.0, 63.5)
- added R25: 10k, Resistor_SMD:R_0603_1608Metric, F.Cu at (193.0, 66.0)
- added R26: 10k, Resistor_SMD:R_0603_1608Metric, F.Cu at (197.0, 58.5)
- added R27: 100k, Resistor_SMD:R_0603_1608Metric, F.Cu at (197.0, 61.0)
- added R28: 2k, Resistor_SMD:R_0603_1608Metric, F.Cu at (197.0, 63.5)
- added R29: 16k, Resistor_SMD:R_0603_1608Metric, F.Cu at (197.0, 66.0)
- added R3: 75R, Resistor_SMD:R_0603_1608Metric, F.Cu at (153.2, 76.0)
- added R31: 0.015R, Resistor_SMD:R_1206_3216Metric, F.Cu at (181.8, 116.2)
- added R32: 100K, Resistor_SMD:R_0603_1608Metric, F.Cu at (161.3, 76.0)
- added R33: 5.1K, Resistor_SMD:R_0603_1608Metric, F.Cu at (165.3, 58.5)
- added R34: 100K, Resistor_SMD:R_0603_1608Metric, F.Cu at (165.3, 61.0)
- added R35: 100K, Resistor_SMD:R_0603_1608Metric, F.Cu at (165.3, 63.5)
- added R36: 100K, Resistor_SMD:R_0603_1608Metric, F.Cu at (165.3, 66.0)
- added R37: 10K, Resistor_SMD:R_0603_1608Metric, F.Cu at (165.3, 68.5)
- added R38: 100K, Resistor_SMD:R_0603_1608Metric, F.Cu at (165.3, 71.0)
- added R39: 10k, Resistor_SMD:R_0603_1608Metric, F.Cu at (165.3, 73.5)
- added R4: 75R, Resistor_SMD:R_0603_1608Metric, F.Cu at (157.2, 58.5)
- added R40: 100K, Resistor_SMD:R_0603_1608Metric, F.Cu at (165.3, 76.0)
- added R5: 75R, Resistor_SMD:R_0603_1608Metric, F.Cu at (157.2, 61.0)
- added R6: 75R, Resistor_SMD:R_0603_1608Metric, F.Cu at (157.2, 63.5)
- added R7: 10k, Resistor_SMD:R_0603_1608Metric, F.Cu at (157.2, 66.0)
- added R8: 10k, Resistor_SMD:R_0603_1608Metric, F.Cu at (157.2, 68.5)
- added R9: 10k, Resistor_SMD:R_0603_1608Metric, F.Cu at (157.2, 71.0)
- added SW1: DSHP03TS-S, ThingsGate-1:SW-SMD_DSHP03TS-S, F.Cu at (170.5, 41.3)
- added T1: H1102NL, ThingsGate-1:H1102NL, F.Cu at (174.2, 62.8)
- added U1: CH334R, Package_SO:QSOP-16_3.9x4.9mm_P0.635mm, F.Cu at (178.4, 49.1)
- added U10: TPS54331DR, ThingsGate-1:TPS54331DDAR_PowerPAD, F.Cu at (124.2, 122.7)
- added U11: RJ45-202-007-02, ThingsGate-1:RJ45-TH_RJ45-202-007-02, F.Cu at (161.3, 106.5)
- added U12: LM74700, Package_TO_SOT_SMD:SOT-23-6, F.Cu at (139.5, 104.4)
- added U13: LM74700, Package_TO_SOT_SMD:SOT-23-6, F.Cu at (139.5, 109.1)
- added U14: LM324, Package_SO:SOIC-14_3.9x8.7mm_P1.27mm, F.Cu at (147.4, 115.4)
- added U15: TF-123B-ARP9H17, ThingsGate-1:TF-SMD_TF-123-ARP9H15, F.Cu at (160.9, 40.0)
- added U2: ThingsCore-1, ThingsGate-1:ThingsCore-1, F.Cu at (123.5, 29.4)
- added U3: POE_PD_Module, ThingsGate-1:SDAPO_DP9700, F.Cu at (121.3, 112.3)
- added U4: LM74700, Package_TO_SOT_SMD:SOT-23-6, F.Cu at (139.5, 99.8)
- added U5: BQ24650, ThingsGate-1:Texas_RVA_VQFN-16-1EP_3.5x3.5mm_P0.5mm_EP2.14x2.14mm_ThermalVias, F.Cu at (202.8, 79.0)
- added U6: TCA9535PWR, Package_SO:SSOP-24_5.3x8.2mm_P0.65mm, F.Cu at (179.1, 40.7)
- added U7: mPCIE-52P-SLOT, ThingsGate-1:mpcie-slot_full, F.Cu at (157.6, 29.4)
- added U8: mPCIE-52P-SLOT, ThingsGate-1:mpcie-slot_full, F.Cu at (191.7, 29.4)
- added U9: TPS54331DR, ThingsGate-1:TPS54331DDAR_PowerPAD, F.Cu at (124.2, 116.3)

Commit message: placement ok
Parts:
- removed R21, R22: 10k, Resistor_SMD:R_0603_1608Metric
- added BT1: S8411-45R, ThingsGate-1:Battery_Holder_CR1220_S8411-45R, F.Cu at (96.8, 26.5)
- added C43: 100n, Capacitor_SMD:C_0603_1608Metric, B.Cu at (82.0, 92.2)
- added C44: 100n, Capacitor_SMD:C_0603_1608Metric, B.Cu at (84.0, 92.2)
- added C45: 100n, Capacitor_SMD:C_0603_1608Metric, B.Cu at (51.5, 45.2)
- added C46: 22u, Capacitor_SMD:C_0805_2012Metric, B.Cu at (22.0, 61.5)
- added C47: 22u, Capacitor_SMD:C_0805_2012Metric, B.Cu at (104.6, 89.0)
- added C48: 22u, Capacitor_SMD:C_0805_2012Metric, B.Cu at (102.3, 89.0)
- added C49: 100n, Capacitor_SMD:C_0603_1608Metric, B.Cu at (75.5, 46.2)
- added C50: 1u, Fuse:Fuse_0805_2012Metric, B.Cu at (76.8, 48.8)
- added C51: 10u, Fuse:Fuse_0805_2012Metric, B.Cu at (74.5, 48.8)
- added C52: 100n, Capacitor_SMD:C_0603_1608Metric, B.Cu at (72.2, 18.8)
- added C53: 1u, Fuse:Fuse_0805_2012Metric, B.Cu at (72.4, 16.8)
- added C54: 100n, Capacitor_SMD:C_0603_1608Metric, B.Cu at (41.5, 24.8)
- added C55: 39p, Capacitor_SMD:C_0603_1608Metric, B.Cu at (39.8, 29.0)
- added C56: 39p, Capacitor_SMD:C_0603_1608Metric, B.Cu at (37.8, 29.0)
- added C57: 39p, Capacitor_SMD:C_0603_1608Metric, B.Cu at (35.8, 29.0)
- added D12: RED, LED_SMD:LED_0603_1608Metric, F.Cu at (21.5, 19.5)
- added F5: 500mA, Fuse:Fuse_1206_3216Metric, B.Cu at (103.6, 92.0)
- added F6: 500mA, Fuse:Fuse_1206_3216Metric, B.Cu at (103.6, 94.8)
- added F7: 500mA, Fuse:Fuse_1206_3216Metric, B.Cu at (22.0, 57.0)
- added G***: LOGO, LOGO, F.Cu at (96.8, 88.2)
- added J1: Conn_02x07_Odd_Even, Connector_IDC:IDC-Header_2x07_P2.54mm_Vertical, F.Cu at (16.7, 27.4)
- added R30: 10k, Resistor_SMD:R_0603_1608Metric, B.Cu at (67.2, 103.5)
- added R41: 10k, Resistor_SMD:R_0603_1608Metric, B.Cu at (65.5, 103.5)
- added R42: 10k, Resistor_SMD:R_0603_1608Metric, B.Cu at (63.8, 103.5)
- added R43: 10k, Resistor_SMD:R_0603_1608Metric, B.Cu at (50.7, 42.8)
- added R44: 10k, Resistor_SMD:R_0603_1608Metric, B.Cu at (50.8, 41.0)
- added R45: 100R, Resistor_SMD:R_0603_1608Metric, B.Cu at (21.8, 39.8)
- added R46: 10k, Resistor_SMD:R_0603_1608Metric, B.Cu at (72.2, 62.0)
- added R47: 10k, Resistor_SMD:R_0603_1608Metric, B.Cu at (51.5, 38.8)
- added R48: 10k, Resistor_SMD:R_0603_1608Metric, B.Cu at (39.2, 62.0)
- added R49: 10k, Resistor_SMD:R_0603_1608Metric, B.Cu at (47.2, 62.0)
- added R50: 10k, Resistor_SMD:R_0603_1608Metric, B.Cu at (69.5, 18.0)
- added R51: 10k, Resistor_SMD:R_0603_1608Metric, B.Cu at (73.0, 22.0)
- added R52: 10k, Resistor_SMD:R_0603_1608Metric, B.Cu at (33.0, 25.5)
- added R53: 0R, Resistor_SMD:R_0603_1608Metric, B.Cu at (30.5, 61.9)
- added R54: 0R, Resistor_SMD:R_0603_1608Metric, B.Cu at (33.2, 62.0)
- added R55: 10k, Resistor_SMD:R_0603_1608Metric, B.Cu at (25.8, 86.3)
- added R56: 10k, Resistor_SMD:R_0603_1608Metric, B.Cu at (25.8, 79.6)
- added R57: 10k, Resistor_SMD:R_0603_1608Metric, B.Cu at (15.8, 77.2)
- added R58: 10k, Resistor_SMD:R_0603_1608Metric, B.Cu at (15.6, 91.2)
- added U16: SMN-305-ARP7, ThingsGate-1:NANO-SIM-SMD_SMN-305-ARP7, F.Cu at (39.0, 20.0)
- added U17: PC817, Package_DIP:DIP-4_W7.62mm_SMDSocket_SmallPads, B.Cu at (19.5, 87.5)
- added U18: PC817, Package_DIP:DIP-4_W7.62mm_SMDSocket_SmallPads, B.Cu at (19.5, 81.0)
- added Y1: X322512MOB4SI, Crystal:Crystal_SMD_3225-4Pin_3.2x2.5mm, B.Cu at (72.8, 42.8)
- C1, C11, C12, C13, C14, C15, C16, C17, C18, C19, C2, C20, C21, C22, C23, C24, C25, C26, C27, C28, C29, C3, C30, C31, C32, C33, C34, C35, C36, C37, C38, C39, C4, C40, C41, C42, C5, C6, C7, C8, D1, D10, D11, D2, D3, D4, D5, D6, D7, D8, D9, F1, F2, F3, F4, L1, L2, L3, L4, Q1, Q2, Q3, Q4, Q5, Q6, Q7, R1, R10, R11, R12, R13, R14, R15, R16, R17, R18, R19, R2, R20, R23, R24, R25, R26, R27, R28, R29, R3, R31, R32, R33, R34, R35, R36, R37, R38, R39, R4, R40, R5, R6, R7, R8, R9, U1, U10, U12, U13, U14, U4, U5, U6, U9: moved to B.Cu
- J7: footprint ThingsGate-1:USB_TYPE_A -> ThingsGate-1:USB-A-TH_AF-ZJB13.7
- moved R19 171.6 mm to (32.0, 83.2), turned to -90 degrees
- moved D8 171.4 mm to (36.8, 80.6), turned to -90 degrees
- moved R26 170.9 mm to (27.2, 78.0), turned to -90 degrees
- moved R29 169.9 mm to (27.2, 72.2), turned to 90 degrees
- moved U5 169.0 mm to (33.8, 77.3), turned to 90 degrees
- moved C37 168.5 mm to (29.2, 75.2), turned to 180 degrees
- moved R28 168.2 mm to (29.0, 72.2), turned to -90 degrees
- moved R27 166.6 mm to (30.8, 72.2), turned to 90 degrees
- moved R23 165.4 mm to (29.0, 82.2)
- moved R24 164.9 mm to (29.0, 80.5)
- moved C33 163.5 mm to (34.5, 82.8), turned to -90 degrees
- moved R25 163.2 mm to (30.2, 78.0), turned to 90 degrees
- moved C35 162.3 mm to (35.4, 73.8), turned to 180 degrees
- moved C38 161.3 mm to (29.0, 84.0)
- moved R31 160.9 mm to (21.8, 99.5), turned to 90 degrees
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Connections:
- C35 pad 1: /Power Harvester/REGN -> GND
- C35 pad 2: GND -> /Power Harvester/REGN
- C40 pad 2: /Power Supply/S_AMP_LP -> CS_AMP_LP
- C41 pad 2: /Power Supply/BUS_VSENSE_LP -> BUS_VSENSE_LP
- C42 pad 2: /Power Supply/BAT_VSENSE_LP -> BAT_VSENSE_LP
- D10 pad 2: /Power Supply/BUS_VSENSE_LP -> BUS_VSENSE_LP
- D11 pad 2: /Power Supply/BAT_VSENSE_LP -> BAT_VSENSE_LP
- D9 pad 2: /Power Supply/S_AMP_LP -> CS_AMP_LP
- J5 pad 1: unconnected-(J5-VBUS1-Pad1) -> /Modules/USB_VB1
- J5 pad 2: unconnected-(J5-D1--Pad2) -> /Modules/USB_P1-
- J5 pad 3: unconnected-(J5-D1+-Pad3) -> /Modules/USB_P1+
- J5 pad 4: unconnected-(J5-GND1-Pad4) -> GND
- J5 pad 5: unconnected-(J5-VBUS2-Pad5) -> /Modules/USB_VB2
- J5 pad 6: unconnected-(J5-D2--Pad6) -> /Modules/USB_P2-
- J5 pad 7: unconnected-(J5-D2+-Pad7) -> /Modules/USB_P2+
- J5 pad 8: unconnected-(J5-GND2-Pad8) -> GND
- J5 pad 9: unconnected-(J5-Shield-Pad9) -> GND
- J7 pad 1: unconnected-(J7-VBUS-Pad1) -> /Modules/USB_OTG_VB1
- J7 pad 2: unconnected-(J7-D--Pad2) -> /Modules/USB2_OTG-
- J7 pad 3: unconnected-(J7-D+-Pad3) -> /Modules/USB2_OTG+
- J7 pad 4: unconnected-(J7-GND-Pad4) -> GND
- J7 pad 5: unconnected-(J7-Shield-Pad5) -> GND
- R32 pad 2: /Power Supply/S_AMP_LP -> CS_AMP_LP
- R35 pad 2: /Power Supply/BUS_VSENSE_LP -> BUS_VSENSE_LP
- R40 pad 2: /Power Supply/BAT_VSENSE_LP -> BAT_VSENSE_LP
- R7 pad 1: LED2 -> ETH_LED2
- R8 pad 1: LED1 -> ETH_LED1
- SW1 pad 1: unconnected-(SW1-Pad1) -> GND
- SW1 pad 2: unconnected-(SW1-Pad2) -> GND
- SW1 pad 3: unconnected-(SW1-Pad3) -> GND
- SW1 pad 4: unconnected-(SW1-Pad4) -> /Modules/BOOT2
- SW1 pad 5: unconnected-(SW1-Pad5) -> /Modules/BOOT1
- SW1 pad 6: unconnected-(SW1-Pad6) -> /Modules/BOOT0
- T1 pad 1: unconnected-(T1-TD+-Pad1) -> ETH_TXP
- T1 pad 2: unconnected-(T1-CT1-Pad2) -> /Power Supply/CT_ETH_PHY
- T1 pad 3: unconnected-(T1-TD--Pad3) -> ETH_TXN
- T1 pad 6: unconnected-(T1-RD+-Pad6) -> ETH_RXP
- T1 pad 7: unconnected-(T1-CT2-Pad7) -> /Power Supply/CT_ETH_PHY
- T1 pad 8: unconnected-(T1-RD--Pad8) -> ETH_RXN
- U1 pad 1: unconnected-(U1-DM4--Pad1) -> /Modules/USB_P1-
- U1 pad 10: unconnected-(U1-DMU--Pad10) -> /Modules/USB1_H-
- U1 pad 11: unconnected-(U1-DPU+-Pad11) -> /Modules/USB1_H+
- U1 pad 12: unconnected-(U1-V5-Pad12) -> 5V
- U1 pad 13: unconnected-(U1-VDD33-Pad13) -> /Modules/HUB_VDD33
- U1 pad 14: unconnected-(U1-GND-Pad14) -> GND
- U1 pad 15: unconnected-(U1-XO-Pad15) -> /Modules/HUB_XO
- U1 pad 16: unconnected-(U1-XI-Pad16) -> /Modules/HUB_XI
- U1 pad 2: unconnected-(U1-DP4+-Pad2) -> /Modules/USB_P1+
- U1 pad 3: unconnected-(U1-DM3--Pad3) -> /Modules/USB_P2-
- U1 pad 4: unconnected-(U1-DP3+-Pad4) -> /Modules/USB_P2+
- U1 pad 5: unconnected-(U1-DM2--Pad5) -> /Modules/LWUSB_D-
- U1 pad 6: unconnected-(U1-DP2+-Pad6) -> /Modules/LWUSB_D+
- U1 pad 7: unconnected-(U1-DM1--Pad7) -> /Modules/LTE_USB_D-
- U1 pad 8: unconnected-(U1-DP1+-Pad8) -> /Modules/LTE_USB_D+
- U14 pad 2: GND -> /Power Supply/S_AMP_P
- U14 pad 3: /Power Supply/S_AMP_P -> GND
- U15 pad 10: unconnected-(U15-SHLD-Pad10) -> GND
- U15 pad 11: unconnected-(U15-SHLD-Pad11) -> GND
- U15 pad 12: unconnected-(U15-SHLD-Pad12) -> GND
- U15 pad 13: unconnected-(U15-SHLD-Pad13) -> GND
- U15 pad 2: unconnected-(U15-CD/DAT3-Pad2) -> /Modules/SD_CS
- U15 pad 3: unconnected-(U15-SDI/CMD-Pad3) -> /Modules/SPI4_MOSI
- U15 pad 4: unconnected-(U15-VDD-Pad4) -> 3V3
- U15 pad 5: unconnected-(U15-CLK-Pad5) -> /Modules/SPI4_SCK
- U15 pad 6: unconnected-(U15-VSS-Pad6) -> GND
- U15 pad 7: unconnected-(U15-SDO/DAT0-Pad7) -> /Modules/SPI4_MISO
- U15 pad 9: unconnected-(U15-CD-Pad9) -> /Modules/SD_DET
- U2 pad 1: unconnected-(U2-ETH_LED2-Pad1) -> ETH_LED2
- U2 pad 10: unconnected-(U2-5VIN-Pad10) -> 5V
- U2 pad 11: unconnected-(U2-ETH_TXN-Pad11) -> ETH_TXN
- U2 pad 12: unconnected-(U2-5VIN-Pad12) -> 5V
- U2 pad 13: unconnected-(U2-UART4_RX-Pad13) -> /Modules/UART4_RX
- U2 pad 15: unconnected-(U2-I2C1_SDA-Pad15) -> /Modules/I2C1_SDA
- U2 pad 16: unconnected-(U2-SPI4_MISO-Pad16) -> /Modules/SPI4_MISO
- U2 pad 17: unconnected-(U2-SPI4_SCK-Pad17) -> /Modules/SPI4_SCK
- U2 pad 18: unconnected-(U2-ADC2_IN3-Pad18) -> CS_AMP_LP
- U2 pad 19: unconnected-(U2-SPI4_MOSI-Pad19) -> /Modules/SPI4_MOSI
- U2 pad 2: unconnected-(U2-GND-Pad2) -> GND
- U2 pad 20: unconnected-(U2-ADC1_IN6-Pad20) -> BUS_VSENSE_LP
- U2 pad 22: unconnected-(U2-ADC2_IN0-Pad22) -> BAT_VSENSE_LP
- U2 pad 25: unconnected-(U2-UART4_TX-Pad25) -> /Modules/UART4_TX
- U2 pad 27: unconnected-(U2-I2C1_SCL-Pad27) -> /Modules/I2C1_SCL
- U2 pad 29: unconnected-(U2-FDCAN1_RX-Pad29) -> /Modules/IO_EXP_~{INT}
- U2 pad 3: unconnected-(U2-ETH_LED1-Pad3) -> ETH_LED1
- U2 pad 30: unconnected-(U2-GND-Pad30) -> GND
- U2 pad 31: unconnected-(U2-FDCAN1_TX-Pad31) -> /Modules/SX1301_CSN
- U2 pad 32: unconnected-(U2-VBAT-Pad32) -> VBAT_SOM
- U2 pad 34: unconnected-(U2-DBG_JTCK-Pad34) -> /Modules/SOM_JTCK
- U2 pad 36: unconnected-(U2-DBG_JTDI-Pad36) -> /Modules/SOM_JTDI
- U2 pad 38: unconnected-(U2-DBG_JTDO-Pad38) -> /Modules/SOM_JTDO
- U2 pad 4: unconnected-(U2-GND-Pad4) -> GND
- U2 pad 40: unconnected-(U2-DBG_JTMS-Pad40) -> /Modules/SOM_JTMS
- U2 pad 41: unconnected-(U2-GND-Pad41) -> GND
- U2 pad 42: unconnected-(U2-+3V3_OUT-Pad42) -> 3V3_SOM
- U2 pad 43: unconnected-(U2-USB2_P-Pad43) -> /Modules/USB2_OTG+
- U2 pad 45: unconnected-(U2-USB2_N-Pad45) -> /Modules/USB2_OTG-
- U2 pad 46: unconnected-(U2-BOOT0-Pad46) -> /Modules/BOOT0
- U2 pad 47: unconnected-(U2-GND-Pad47) -> GND
- U2 pad 48: unconnected-(U2-BOOT1-Pad48) -> /Modules/BOOT1
- U2 pad 49: unconnected-(U2-USB1_P-Pad49) -> /Modules/USB1_H+
- U2 pad 5: unconnected-(U2-ETH_RXP-Pad5) -> ETH_RXP
- U2 pad 50: unconnected-(U2-BOOT2-Pad50) -> /Modules/BOOT2
- U2 pad 51: unconnected-(U2-USB1_N-Pad51) -> /Modules/USB1_H-
- U2 pad 52: unconnected-(U2-NRST-Pad52) -> /Modules/SOM_NRST
- U2 pad 6: unconnected-(U2-GND-Pad6) -> GND
- U2 pad 7: unconnected-(U2-ETH_RXN-Pad7) -> ETH_RXN
- U2 pad 8: unconnected-(U2-5VIN-Pad8) -> 5V
- U2 pad 9: unconnected-(U2-ETH_TXP-Pad9) -> ETH_TXP
- U2 pad S1: unconnected-(U2-PadS1) -> GND
- U2 pad S2: unconnected-(U2-PadS2) -> GND
- U5 pad 3: HARV_STAT1 -> /Power Harvester/STAT1
- U5 pad 5: HARV_STAT2 -> /Power Harvester/STAT2
- U6 pad 1: unconnected-(U6-~{INT}-Pad1) -> /Modules/IO_EXP_~{INT}
- U6 pad 10: unconnected-(U6-P06-Pad10) -> /Modules/MCU_NRST
- U6 pad 11: unconnected-(U6-P07-Pad11) -> /Modules/SX1261_NRST_LTE
- U6 pad 12: unconnected-(U6-GND-Pad12) -> GND
- U6 pad 13: unconnected-(U6-P10-Pad13) -> /Modules/MCU_NRST_LTE
- U6 pad 2: unconnected-(U6-A1-Pad2) -> GND
- U6 pad 21: unconnected-(U6-A0-Pad21) -> GND
- U6 pad 22: unconnected-(U6-SCL-Pad22) -> /Modules/I2C1_SCL
- U6 pad 23: unconnected-(U6-SDA-Pad23) -> /Modules/I2C1_SDA
- U6 pad 24: unconnected-(U6-VCC-Pad24) -> 3V3
- U6 pad 3: unconnected-(U6-A2-Pad3) -> GND
- U6 pad 4: unconnected-(U6-P00-Pad4) -> HARV_STAT1
- U6 pad 5: unconnected-(U6-P01-Pad5) -> HARV_STAT2
- U6 pad 6: unconnected-(U6-P02-Pad6) -> /Modules/LW_RST
- U6 pad 7: unconnected-(U6-P03-Pad7) -> /Modules/SD_DET
- U6 pad 8: unconnected-(U6-P04-Pad8) -> /Modules/LTE_RST
- U6 pad 9: unconnected-(U6-P05-Pad9) -> /Modules/SX1261_NRST
- U7 pad 10: unconnected-(U7-Pad10) -> /Modules/USIM_DATA
- U7 pad 11: unconnected-(U7-Pad11) -> Net-(R53-Pad1)
- U7 pad 12: unconnected-(U7-Pad12) -> /Modules/USIM_CLK
- U7 pad 13: unconnected-(U7-Pad13) -> Net-(R54-Pad2)
- U7 pad 14: unconnected-(U7-Pad14) -> /Modules/USIM_RST
- U7 pad 15: unconnected-(U7-Pad15) -> GND
- U7 pad 18: unconnected-(U7-Pad18) -> GND
- U7 pad 2: unconnected-(U7-Pad2) -> 3V3
- U7 pad 21: unconnected-(U7-Pad21) -> GND
- U7 pad 22: unconnected-(U7-Pad22) -> /Modules/LTE_RST
- U7 pad 26: unconnected-(U7-Pad26) -> GND
- U7 pad 27: unconnected-(U7-Pad27) -> GND
- U7 pad 29: unconnected-(U7-Pad29) -> GND
- U7 pad 30: unconnected-(U7-Pad30) -> /Modules/I2C1_SCL
- U7 pad 32: unconnected-(U7-Pad32) -> /Modules/I2C1_SDA
- U7 pad 34: unconnected-(U7-Pad34) -> GND
- U7 pad 35: unconnected-(U7-Pad35) -> GND
- U7 pad 36: unconnected-(U7-Pad36) -> /Modules/LTE_USB_D-
- U7 pad 37: unconnected-(U7-Pad37) -> GND
- U7 pad 38: unconnected-(U7-Pad38) -> /Modules/LTE_USB_D+
- U7 pad 39: unconnected-(U7-Pad39) -> 3V3
- U7 pad 4: unconnected-(U7-Pad4) -> GND
- U7 pad 40: unconnected-(U7-Pad40) -> GND
- U7 pad 41: unconnected-(U7-Pad41) -> 3V3
- U7 pad 42: unconnected-(U7-Pad42) -> /Modules/LED_WWAN
- U7 pad 43: unconnected-(U7-Pad43) -> GND
- U7 pad 44: unconnected-(U7-Pad44) -> /Modules/USIM_DET
- U7 pad 50: unconnected-(U7-Pad50) -> GND
- U7 pad 52: unconnected-(U7-Pad52) -> 3V3
- U7 pad 8: unconnected-(U7-Pad8) -> /Modules/USIM_VDD
- U7 pad 9: unconnected-(U7-Pad9) -> GND
- U7 pad S1: unconnected-(U7-PadS1) -> GND
- U7 pad S2: unconnected-(U7-PadS2) -> GND
- U8 pad 11: unconnected-(U8-Pad11) -> /Modules/SX1261_NRST
- U8 pad 13: unconnected-(U8-Pad13) -> /Modules/MCU_NRST
- U8 pad 15: unconnected-(U8-Pad15) -> GND
- U8 pad 18: unconnected-(U8-Pad18) -> GND
- U8 pad 2: unconnected-(U8-Pad2) -> 3V3
- U8 pad 21: unconnected-(U8-Pad21) -> GND
- U8 pad 22: unconnected-(U8-Pad22) -> /Modules/LW_RST
- U8 pad 24: unconnected-(U8-Pad24) -> 3V3
- U8 pad 26: unconnected-(U8-Pad26) -> GND
- U8 pad 27: unconnected-(U8-Pad27) -> GND
- U8 pad 29: unconnected-(U8-Pad29) -> GND
- U8 pad 30: unconnected-(U8-Pad30) -> /Modules/I2C1_SCL
- U8 pad 32: unconnected-(U8-Pad32) -> /Modules/I2C1_SDA
- U8 pad 34: unconnected-(U8-Pad34) -> GND
- U8 pad 35: unconnected-(U8-Pad35) -> GND
- U8 pad 36: unconnected-(U8-Pad36) -> /Modules/LWUSB_D-
- U8 pad 37: unconnected-(U8-Pad37) -> GND
- U8 pad 38: unconnected-(U8-Pad38) -> /Modules/LWUSB_D+
- U8 pad 39: unconnected-(U8-Pad39) -> 3V3
- U8 pad 4: unconnected-(U8-Pad4) -> GND
- U8 pad 40: unconnected-(U8-Pad40) -> GND
- U8 pad 41: unconnected-(U8-Pad41) -> 3V3
- U8 pad 43: unconnected-(U8-Pad43) -> GND
- U8 pad 45: unconnected-(U8-Pad45) -> /Modules/SPI4_SCK
- U8 pad 47: unconnected-(U8-Pad47) -> /Modules/SPI4_MOSI
- U8 pad 49: unconnected-(U8-Pad49) -> /Modules/SPI4_MISO
- U8 pad 50: unconnected-(U8-Pad50) -> GND
- U8 pad 51: unconnected-(U8-Pad51) -> /Modules/SX1301_CSN
- U8 pad 52: unconnected-(U8-Pad52) -> 3V3
- U8 pad 9: unconnected-(U8-Pad9) -> GND
- U8 pad S1: unconnected-(U8-PadS1) -> GND
- U8 pad S2: unconnected-(U8-PadS2) -> GND
Routing:
- added copper zone on In1.Cu, net GND
Other:
- board text added: "+"
- board text added: "12V BAT"
- board text added: "12V PSU"
- board text added: "JTAG"
- board text added: "LORAWAN"
- board text added: "LTE"
- board text added: "NET"
- board text added: "OTG"
- board text added: "POE"
- board text added: "RTC"
- board text added: "SD"
- board text added: "SIM"
- board text added: "SOLAR"
- board text added: "THINGSGATE-l"

Commit message: layout finished. checks and fab files remaining
Parts:
- moved R49 6.50 mm to (47.0, 55.5)
- moved F4 4.44 mm to (101.0, 64.7)
- moved L4 4.07 mm to (104.5, 65.9), turned to 90 degrees
- moved R30 3.45 mm to (63.8, 103.5)
- moved R42 3.45 mm to (67.2, 103.5)
- moved F6 2.65 mm to (103.5, 92.1)
- moved F5 2.61 mm to (103.5, 94.6)
- moved C8 2.41 mm to (104.0, 63.4), turned to 0 degrees
- moved D7 1.39 mm to (102.2, 69.1), turned to 180 degrees
- moved D6 1.25 mm to (29.6, 92.6), turned to 90 degrees
- moved R2 1.24 mm to (31.9, 90.7), turned to 90 degrees
- moved R46 1.20 mm to (72.2, 63.2)
- moved U3 0.95 mm to (107.8, 19.6)
- moved T1 0.89 mm to (79.9, 93.9)
- moved C22 0.65 mm to (79.0, 93.7)
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Connections:
- H1 pad 1: unconnected-(H1-Pad1) -> CHASSIS
- H2 pad 1: unconnected-(H2-Pad1)_2 -> CHASSIS
- H3 pad 1: unconnected-(H3-Pad1) -> CHASSIS
- H4 pad 1: unconnected-(H4-Pad1)_1 -> CHASSIS
- J5 pad 9: GND -> CHASSIS
- J7 pad 5: GND -> CHASSIS
- SW1 pad 4: /Modules/BOOT2 -> /Modules/BOOT0
- SW1 pad 6: /Modules/BOOT0 -> /Modules/BOOT2
- U6 pad 11: /Modules/SX1261_NRST_LTE -> /Modules/SX1261_NRST
- U6 pad 13: /Modules/MCU_NRST_LTE -> /Modules/SX1261_NRST_LTE
- U6 pad 14: unconnected-(U6-P11-Pad14) -> /Modules/MCU_NRST_LTE
- U6 pad 4: HARV_STAT1 -> unconnected-(U6-P00-Pad4)
- U6 pad 6: /Modules/LW_RST -> HARV_STAT1
- U6 pad 7: /Modules/SD_DET -> /Modules/LTE_RST
- U6 pad 8: /Modules/LTE_RST -> /Modules/SD_DET
- U6 pad 9: /Modules/SX1261_NRST -> /Modules/LW_RST
Routing:
- net CHASSIS: track 0.00 -> 312.6 mm, vias 0 -> 1
- net 5V: track 0.00 -> 287.3 mm, vias 0 -> 32
- net GND: track 0.00 -> 147.4 mm, vias 0 -> 249
- net 12VPOE: track 0.00 -> 135.9 mm
- net /Modules/SPI4_MOSI: track 0.00 -> 120.9 mm, vias 0 -> 2
- net /Modules/UART4_RX: track 0.00 -> 117.3 mm, vias 0 -> 1
- net /Power Supply/VA1: track 0.00 -> 116.6 mm, vias 0 -> 2
- net /Modules/SPI4_SCK: track 0.00 -> 116.2 mm, vias 0 -> 2
- net /Modules/SOM_JTMS: track 0.00 -> 115.0 mm
- net /Modules/USB_P2-: track 0.00 -> 113.4 mm, vias 0 -> 1
- net /Power Supply/VB1: track 0.00 -> 112.6 mm, vias 0 -> 2
- net /Modules/SOM_JTCK: track 0.00 -> 112.3 mm
- net /Power Supply/VB2: track 0.00 -> 112.2 mm, vias 0 -> 2
- net /Power Supply/VA2: track 0.00 -> 111.6 mm, vias 0 -> 2
- net /Modules/USB_P2+: track 0.00 -> 111.0 mm, vias 0 -> 1
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- added copper zone on B.Cu, net /Modules/USB_OTG_VB1
- added copper zone on B.Cu, net /Power Harvester/D_HARV
- added copper zone on B.Cu, net /Power Harvester/SRP
- added copper zone on B.Cu, net /Power Harvester/VCC_HARV
- added copper zone on B.Cu, net /Power Harvester/VREF_HARV
- added copper zone on B.Cu, net /Power Supply/12VBAT_CONN
- added copper zone on B.Cu, net /Power Supply/12VPSU_CONN
- added copper zone on B.Cu, net /Power Supply/3V3_PH
- added copper zone on B.Cu, net /Power Supply/5V_PH
- added copper zone on B.Cu, net /Power Supply/VDC_POE
- added copper zone on B.Cu, net /Power Supply/VSOL_CONN
- added copper zone on B.Cu, net /Power Supply/VSOL_SENSE
- added copper zone on B.Cu, net 12VBAT
- added copper zone on B.Cu, net 12VBAT_HARV
- added copper zone on B.Cu, net 12VPOE
- added copper zone on B.Cu, net 12VPSU
- added copper zone on B.Cu, net 3V3
- added copper zone on F.Cu, net 3V3
- added copper zone on In1.Cu, net 3V3
- added copper zone on B.Cu, net 5V
- added copper zone on F.Cu, net 5V
- added copper zone on In1.Cu, net 5V
- added copper zone on B.Cu, net GND
- added copper zone on F.Cu, net GND
- added copper zone on In2.Cu, net GND
- added copper zone on B.Cu, net Net-(C8-Pad1)
- added copper zone on B.Cu, net VBUS
- added copper zone on B.Cu, net VBUS_FUSE
- added copper zone on F.Cu, net VBUS_FUSE
- added copper zone on B.Cu, net VSOL
- removed copper zone on In1.Cu, net GND
Other:
- board text added: "DESIGNED BY"
- board text added: "LORA MODEM"
- board text added: "PATSAOGLOU P."
- board text added: "REV 1"
- board text removed: "LORAWAN"

Commit message: final fab files and checks done
Parts:
- added C58: 10u, Fuse:Fuse_0805_2012Metric, B.Cu at (36.1, 87.4)
- added TP1: TestPoint, TestPoint:TestPoint_Pad_D1.5mm, F.Cu at (91.9, 59.3)
- added TP2: TestPoint, TestPoint:TestPoint_Pad_D1.5mm, F.Cu at (71.5, 86.7)
- added TP3: TestPoint, TestPoint:TestPoint_Pad_D1.5mm, F.Cu at (102.5, 80.7)
- added TP4: TestPoint, TestPoint:TestPoint_Pad_D1.5mm, F.Cu at (104.4, 89.9)
- added TP5: TestPoint, TestPoint:TestPoint_Pad_D1.5mm, F.Cu at (104.1, 92.4)
- added TP6: TestPoint, TestPoint:TestPoint_Pad_D1.5mm, F.Cu at (15.7, 102.5)
- added TP7: TestPoint, TestPoint:TestPoint_Pad_D1.5mm, F.Cu at (17.0, 49.5)
- added TP8: TestPoint, TestPoint:TestPoint_Pad_D1.5mm, F.Cu at (20.6, 49.5)
- C7: footprint Capacitor_SMD:C_0603_1608Metric -> Capacitor_SMD:C_1206_3216Metric
- moved R5 1.60 mm to (81.4, 98.0)
- moved R3 1.25 mm to (79.9, 98.0)
- moved C7 1.05 mm to (84.8, 97.7)
- moved R4 0.75 mm to (78.5, 98.0)
- moved R6 0.25 mm to (77.0, 98.0)
Connections:
- U2 pad 44: unconnected-(U2-PWR_ONRST-Pad44) -> /Modules/PWR_ONRST
Routing:
- net /Modules/PWR_ONRST: track 0.00 -> 85.2 mm
- net 12VBAT_HARV: track 62.4 -> 93.4 mm, vias 3 -> 4
- net /Modules/SOM_NRST: track 106.5 -> 98.6 mm
- net 12VPOE: track 135.9 -> 139.9 mm, vias 0 -> 1
- net /Modules/UART4_TX: track 110.8 -> 106.9 mm
- net /Modules/UART4_RX: track 117.3 -> 114.5 mm
- net VBUS_FUSE: track 4.53 -> 6.73 mm
- net 3V3: track 43.2 -> 45.3 mm
- net Net-(C7-Pad2): track 7.62 -> 5.77 mm
- net /Power Supply/VA2: track 111.6 -> 112.9 mm
- net BUS_VSENSE_LP: track 60.0 -> 61.1 mm
- net /Power Harvester/STAT1: track 20.9 -> 21.8 mm
- net 3V3_SOM: track 107.5 -> 106.6 mm
- net /Power Supply/VSOL_SENSE: track 78.4 -> 79.1 mm
- net /Modules/SOM_JTDO: track 108.1 -> 107.4 mm
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Other:
- board text added: "12VH"
- board text added: "12VPOE"
- board text added: "3V3"
- board text added: "5V"
- board text added: "NRST"
- board text added: "PWRON"
- board text added: "VBUSF"
